Commit message: coke can works

File: data/toys/white_large_cappuccino_mug.urdf (robot description, URDF)
Before this commit: robot white_large_cappuccino_mug, 1 links, 0 joints
Links:
- link Non-Disposable Cup/Mug: geometry collision mesh filename=white_large_cappuccino_mug_collision.obj scale=1 1 1; visual mesh filename=white_large_cappuccino_mug.obj scale=1 1 1
